Commit message: anymal velocity control to be trained on PC with PPO

File: dflex/dflex/envs/assets/anymal_c/urdf/anymal.urdf (robot description, URDF)
Before this commit: robot anymal, 77 links, 76 joints
Links:
- added link base_inertia, mass 6.222
- link LF_FOOT: geometry collision cylinder length=0.282504 radius=0.0175; collision sphere radius=0.03
- link LF_HFE: geometry collision cylinder length=0.14 radius=0.05; visual mesh filename=../meshes/drive.dae scale=1.0 1.0 1.0
- link LF_KFE: geometry collision cylinder length=0.14 radius=0.05; visual mesh filename=../meshes/drive.dae scale=1.0 1.0 1.0
- link LF_SHANK: geometry 
- link LF_shank_fixed: geometry collision box size=0.114998 0.0675 0.04; collision cylinder length=0.04 radius=0.06
- link LF_thigh_fixed: geometry collision box size=0.075 0.06 0.282627; collision cylinder length=0.08 radius=0.065
- link LH_FOOT: geometry collision cylinder length=0.282504 radius=0.0175; collision sphere radius=0.03
- link LH_HFE: geometry collision cylinder length=0.14 radius=0.05; visual mesh filename=../meshes/drive.dae scale=1.0 1.0 1.0
- link LH_KFE: geometry collision cylinder length=0.14 radius=0.05; visual mesh filename=../meshes/drive.dae scale=1.0 1.0 1.0
- link LH_SHANK: geometry 
- link LH_shank_fixed: geometry collision box size=0.114998 0.0675 0.04; collision cylinder length=0.04 radius=0.06
- link LH_thigh_fixed: geometry collision box size=0.075 0.06 0.282627; collision cylinder length=0.08 radius=0.065
- link RF_FOOT: geometry collision cylinder length=0.282504 radius=0.0175; collision sphere radius=0.03
- link RF_HFE: geometry collision cylinder length=0.14 radius=0.05; visual mesh filename=../meshes/drive.dae scale=1.0 1.0 1.0
- link RF_KFE: geometry collision cylinder length=0.14 radius=0.05; visual mesh filename=../meshes/drive.dae scale=1.0 1.0 1.0
- link RF_SHANK: geometry 
- link RF_shank_fixed: geometry collision box size=0.114998 0.0675 0.04; collision cylinder length=0.04 radius=0.06
- link RF_thigh_fixed: geometry collision box size=0.075 0.06 0.282627; collision cylinder length=0.08 radius=0.065
- link RH_FOOT: geometry collision cylinder length=0.282504 radius=0.0175; collision sphere radius=0.03
- link RH_HFE: geometry collision cylinder length=0.14 radius=0.05; visual mesh filename=../meshes/drive.dae scale=1.0 1.0 1.0
- link RH_KFE: geometry collision cylinder length=0.14 radius=0.05; visual mesh filename=../meshes/drive.dae scale=1.0 1.0 1.0
- link RH_SHANK: geometry 
- link RH_shank_fixed: geometry collision box size=0.114998 0.0675 0.04; collision cylinder length=0.04 radius=0.06
- link RH_thigh_fixed: geometry collision box size=0.075 0.06 0.282627; collision cylinder length=0.08 radius=0.065
- link base: mass 6.222 -> None; geometry collision box size=0.58 0.14 0.18; collision cylinder length=0.145 radius=0.09
- link face_front: geometry collision box size=0.11 0.14 0.18; collision cylinder length=0.11 radius=0.09
- link face_rear: geometry collision box size=0.11 0.14 0.18; collision cylinder length=0.11 radius=0.09
- link imu_link: geometry collision box size=0.024 0.024 0.01; visual box size=0.024 0.024 0.01
- link lidar_cage: geometry collision cylinder length=0.12 radius=0.07; visual mesh filename=../meshes/lidar_cage.dae scale=1.0 1.0 1.0
Joints:
- added joint base_to_base_inertia: type fixed, parent base, child base_inertia, origin xyz=0 0 0 rpy=0 0 0
- joint LF_HAA: limit effort=80.0 velocity=20. -> lower=-0.72 upper=0.49 effort=80.0 velocity=7.5
- joint LF_HFE: limit effort=80.0 velocity=20. -> lower=-9.42477796077 upper=9.42477796077 effort=80.0 velocity=7.5
- joint LF_KFE: limit effort=80.0 velocity=20. -> lower=-9.42477796077 upper=9.42477796077 effort=80.0 velocity=7.5
- joint LH_HAA: limit effort=80.0 velocity=20. -> lower=-0.72 upper=0.49 effort=80.0 velocity=7.5
- joint LH_HFE: limit effort=80.0 velocity=20. -> lower=-9.42477796077 upper=9.42477796077 effort=80.0 velocity=7.5
- joint LH_KFE: limit effort=80.0 velocity=20. -> lower=-9.42477796077 upper=9.42477796077 effort=80.0 velocity=7.5
- joint RF_HAA: limit effort=80.0 velocity=20. -> lower=-0.49 upper=0.72 effort=80.0 velocity=7.5
- joint RF_HFE: limit effort=80.0 velocity=20. -> lower=-9.42477796077 upper=9.42477796077 effort=80.0 velocity=7.5
- joint RF_KFE: limit effort=80.0 velocity=20. -> lower=-9.42477796077 upper=9.42477796077 effort=80.0 velocity=7.5
- joint RH_HAA: limit effort=80.0 velocity=20. -> lower=-0.49 upper=0.72 effort=80.0 velocity=7.5
- joint RH_HFE: limit effort=80.0 velocity=20. -> lower=-9.42477796077 upper=9.42477796077 effort=80.0 velocity=7.5
- joint RH_KFE: limit effort=80.0 velocity=20. -> lower=-9.42477796077 upper=9.42477796077 effort=80.0 velocity=7.5
